Commit message: feat: replace DiffDrive plugin with ros2_control + diff_drive_controller

File: src/rover_description/urdf/rover.urdf.xacro (robot description, xacro)
@@ -1,269 +1,11 @@
 <?xml version="1.0"?>
 <robot xmlns:xacro="http://www.ros.org/wiki/xacro" name="warehouse_rover">
-<xacro:property name="body_length" value="0.80" />
-<xacro:property name="body_width"  value="0.60" />
-<xacro:property name="body_height" value="0.30" />
-<xacro:property name="ground_clearance"  value="0.1" />
-<xacro:property name="wheel_radius" value="0.10" />
-<xacro:property name="wheel_width"  value="0.05" />
-<xacro:property name="wheel_separation" value="0.66" />
-<xacro:property name="caster_radius"  value="0.05" />
-<xacro:property name="body_mass" value="70"/>
-<xacro:property name="wheel_mass" value="2.5"/>
-<xacro:property name="caster_mass" value="1.25"/>
-<xacro:property name="laser_length" value="0.111" />
-<xacro:property name="laser_width"  value="0.112" />
-<xacro:property name="laser_height" value="0.135" />
-<xacro:property name="laser_mass" value="1.15"/>
-<xacro:property name="camera_length" value="0.03" />
-<xacro:property name="camera_width"  value="0.09" />
-<xacro:property name="camera_height" value="0.025" />
-<xacro:property name="camera_mass" value="0.072"/>
-<xacro:property name="deck_height" value="${ ground_clearance + body_height }"/>
-<xacro:property name="base_foot" value="${ (body_height/2) + ground_clearance }"/>
-<xacro:macro name="box_inertia" params="mass x y z">
-  <inertial>
-    <mass value="${mass}"/>
-    <inertia ixx="${mass*(y*y+z*z)/12}" ixy="0" ixz="0"
-             iyy="${mass*(x*x+z*z)/12}" iyz="0"
-             izz="${mass*(x*x+y*y)/12}"/>
-  </inertial>
-</xacro:macro>
-<xacro:macro name="cylinder_inertia" params="mass r h">
-  <inertial>
-    <mass value="${mass}"/>
-    <inertia ixx="${(mass/12)*(3*r*r+h*h)}" ixy="0" ixz="0"
-             iyy="${(mass/2)*(r*r)}" iyz="0"
-             izz="${(mass/12)*(3*r*r+h*h)}"/>
-  </inertial>
-</xacro:macro>
-<xacro:macro name="sphere_inertia" params="mass r">
-  <inertial>
-    <mass value="${mass}"/>
-      <inertia ixx="${(2/5) * mass * (r*r)}" ixy="0" ixz="0"
-             iyy="${(2/5) * mass * (r*r)}" iyz="0"
-             izz="${(2/5) * mass * (r*r)}"/>
-  </inertial>
-</xacro:macro>
-<xacro:macro name="caster_wheel" params="prefix *origin">
-   <link name="${prefix}">
-    <visual>
-      <geometry>
-        <sphere radius="${caster_radius}"/>
-      </geometry>
-    </visual>
-    <collision>
-  <geometry>
-    <sphere radius="${caster_radius}"/>
-  </geometry>
-</collision>
-    <xacro:sphere_inertia mass="${caster_mass}" r="${caster_radius}"/>
-  </link>
-<gazebo reference="${prefix}">
-  <mu1>0.0</mu1>
-  <mu2>0.0</mu2>
-</gazebo>
-  <joint name="${prefix}_joint" type="fixed">
-    <parent link="base_link"/>
-    <child link="${prefix}"/>
-    <xacro:insert_block name="origin"/>
-  </joint>
-</xacro:macro>
-<link name="base_footprint"/>
-<joint name="base_footprint_joint" type="fixed">
-  <parent link="base_footprint"/>
-  <child link="base_link"/>
-  <origin xyz="0 0.0 ${base_foot}" />
-</joint>
-  <link name="base_link">
-    <visual>
-      <geometry>
-        <box size="${body_length} ${body_width} ${body_height} "/>
-      </geometry>
-    </visual>
-    <collision>
-      <geometry>
-        <box size="${body_length} ${body_width} ${body_height}"/>
-      </geometry>
-    </collision>
-    <xacro:box_inertia mass="${body_mass}" x="${body_length}" y="${body_width}" z="${body_height}"/>
-  </link>
-<link name="left_wheel">
-  <visual>
-  <origin rpy="1.57 0 0" xyz="0 0 0"/>
-      <geometry>
-        <cylinder radius="${wheel_radius}" length="${wheel_width}"/>
-      </geometry>
-  </visual>
-  <collision>
-  <origin rpy="1.57 0 0" xyz="0 0 0"/>
-  <geometry>
-    <cylinder radius="${wheel_radius}" length="${wheel_width}"/>
-  </geometry>
-</collision>
-<xacro:cylinder_inertia mass="${wheel_mass}" r="${wheel_radius}" h="${wheel_width}"/>
-</link>
-<joint name="left_wheel_joint" type="continuous">
-  <parent link="base_link"/>
-  <child link="left_wheel"/>
-  <origin xyz="0 ${wheel_separation/2} ${-(body_height/2)}"/>
-  <axis xyz="0 1 0"/>
-</joint>
-<link name="right_wheel">
-  <visual>
-  <origin rpy="1.57 0 0" xyz="0 0 0"/>
-      <geometry>
-        <cylinder radius="${wheel_radius}" length="${wheel_width}"/>
-      </geometry>
-  </visual>
-  <collision>
-  <origin rpy="1.57 0 0" xyz="0 0 0"/>
-  <geometry>
-    <cylinder radius="${wheel_radius}" length="${wheel_width}"/>
-  </geometry>
-</collision>
-<xacro:cylinder_inertia mass="${wheel_mass}" r="${wheel_radius}" h="${wheel_width}"/>
-</link>
-    <gazebo reference="left_wheel">
-      <mu1>1.0</mu1>
-      <mu2>1.0</mu2>
-</gazebo>
-    <gazebo reference="right_wheel">
-      <mu1>1.0</mu1>
-      <mu2>1.0</mu2>
-</gazebo>
-<joint name="right_wheel_joint" type="continuous">
-  <parent link="base_link"/>
-  <child link="right_wheel"/>
-  <origin xyz="0 ${-wheel_separation/2} ${-(body_height/2)}"/>
-  <axis xyz="0 1 0"/>
-</joint>
-<xacro:caster_wheel prefix="caster_front_left">
-  <origin xyz="0.30 0.2 ${caster_radius - (ground_clearance + body_height/2)}"/>
-</xacro:caster_wheel>
-<xacro:caster_wheel prefix="caster_front_right">
-  <origin xyz="0.30 -0.2 ${caster_radius - (ground_clearance + body_height/2)}"/>
-</xacro:caster_wheel>
-<xacro:caster_wheel prefix="caster_rear_left">
-  <origin xyz="-0.30 0.2 ${caster_radius - (ground_clearance + body_height/2)}"/>
-</xacro:caster_wheel>
-<xacro:caster_wheel prefix="caster_rear_right">
-  <origin xyz="-0.30 -0.2 ${caster_radius - (ground_clearance + body_height/2)}"/>
-</xacro:caster_wheel>
-<gazebo>
-  <plugin filename="gz-sim-diff-drive-system"
-          name="gz::sim::systems::DiffDrive">
-    <left_joint>left_wheel_joint</left_joint>
-    <right_joint>right_wheel_joint</right_joint>
-    <wheel_separation>${wheel_separation}</wheel_separation>
-    <wheel_radius>${wheel_radius}</wheel_radius>
-    <topic>cmd_vel</topic>
-    <odom_topic>odom</odom_topic>
-    <frame_id>odom</frame_id>
-    <child_frame_id>base_footprint</child_frame_id>
-  </plugin>
-</gazebo>
-<gazebo>
-  <plugin filename="gz-sim-joint-state-publisher-system"
-          name="gz::sim::systems::JointStatePublisher">
-    <topic>joint_states</topic>
-    <joint_name>left_wheel_joint</joint_name>
-    <joint_name>right_wheel_joint</joint_name>
-  </plugin>
-</gazebo>
-<link name="laser_link">
-  <visual>
-    <geometry>
-      <box size="${laser_length} ${laser_width} ${laser_height}"/>
-    </geometry>
-  </visual>
-  <collision>
-    <geometry>
-      <box size="${laser_length} ${laser_width} ${laser_height}"/>
-    </geometry>
-  </collision>
-  <xacro:box_inertia mass="${laser_mass}" x="${laser_length}" y="${laser_width}" z="${laser_height}" />
-</link>
-<joint name="laser_joint" type="fixed">
-  <origin xyz="${body_length/2 + laser_length/2} 0.0 ${body_height/2 + laser_height/2}"/>
-  <parent link="base_link"/>
-  <child link="laser_link"/>
-</joint>
-<link name="camera_link">
-  <visual>
-    <geometry>
-      <box size="${camera_length} ${camera_width} ${camera_height}"/>
-    </geometry>
-  </visual>
-  <collision>
-    <geometry>
-      <box size="${camera_length} ${camera_width} ${camera_height}"/>
-    </geometry>
-  </collision>
-  <xacro:box_inertia mass="${camera_mass}" x="${camera_length}" y="${camera_width}" z="${camera_height}" />
-</link>
-<joint name="camera_joint" type="fixed">
-  <origin xyz="${laser_length/2 + camera_length/2 } 0.0 ${laser_height/2 + camera_height /2}"/>
-  <parent link="laser_link"/>
-  <child link="camera_link"/>
-</joint>
-<gazebo reference="laser_link">
-  <sensor name="laser" type="gpu_lidar">
-    <topic>scan</topic>
-    <update_rate>10</update_rate>
-    <always_on>true</always_on>
-    <visualize>true</visualize>
-    <lidar>
-      <scan>
-        <horizontal>
-          <samples>705</samples>
-          <resolution>1</resolution>
-          <min_angle>-2.4</min_angle>
-          <max_angle>2.4</max_angle>
-        </horizontal>
-      </scan>
-      <range>
-        <min>0.05</min>
-        <max>9.0</max>
-        <resolution>0.01</resolution>
-      </range>
-    </lidar>
-  </sensor>
-</gazebo>
-<link name="imu_link">
-  <xacro:box_inertia mass="0.05" x="0.02" y="0.02" z="0.01"/>
-</link>
-<joint name="imu_joint" type="fixed">
-  <parent link="base_link"/>
-  <child link="imu_link"/>
-  <origin xyz="0 0 0"/>
-</joint>
-<gazebo reference="imu_link">
-  <sensor name="imu" type="imu">
-    <topic>imu</topic>
-    <update_rate>100</update_rate>
-    <always_on>true</always_on>
-    <gz_frame_id>imu_link</gz_frame_id>
-  </sensor>
-</gazebo>
-<gazebo reference="camera_link">
-  <sensor name="camera" type="camera">
-    <topic>camera/image_raw</topic>
-    <update_rate>30</update_rate>
-    <always_on>true</always_on>
-    <gz_frame_id>camera_link</gz_frame_id>
-    <camera>
-      <horizontal_fov>1.047</horizontal_fov>
-      <image>
-        <width>640</width>
-        <height>480</height>
-        <format>R8G8B8</format>
-      </image>
-      <clip>
-        <near>0.1</near>
-        <far>15.0</far>
-      </clip>
-    </camera>
-  </sensor>
-</gazebo>
+<xacro:include filename="$(find rover_description)/urdf/properties.xacro"/>
+<xacro:include filename="$(find rover_description)/urdf/inertia_macros.xacro"/>
+<xacro:include filename="$(find rover_description)/urdf/base.xacro"/>
+<xacro:include filename="$(find rover_description)/urdf/wheels.xacro"/>
+<xacro:include filename="$(find rover_description)/urdf/ros2_control.xacro"/>
+<xacro:include filename="$(find rover_description)/urdf/caster_wheels.xacro"/>
+<xacro:include filename="$(find rover_description)/urdf/gazebo_links.xacro"/>
+<xacro:include filename="$(find rover_description)/urdf/gazebo_plugins.xacro"/>
 </robot>
